File: hardware/raster-bot/raster-bot.kicad_pcb (KiCad board)
At the start: 2 copper layers, 66 x 45 mm, 37 parts, among them J1 JUMPER_2PIN, J2 JUMPER_2PIN, J3 PinSocket_1x10, J4 JUMPER_2PIN, J5 EYESPI_Connector, J6 PinSocket_2x06, J7 JST_PH, J8 PinSocket_1x02, SW1 SW_SPDT, U1 DRV8833PWPR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

Commit message: PCB v0.2 update - added motor JST connectors; refactored custom footprints
Parts:
- removed the J3 at (122.2, 108.3)
- removed the J6 at (154.1, 105.7)
- added J5: Conn_Motor_N20_Encoder, Connector_JST:JST_SH_BM06B-SRSS-TB_1x06-1MP_P1.00mm_Vertical, F.Cu at (146.6, 107.1)
- added J8: Conn_Motor_N20_Encoder, Connector_JST:JST_SH_BM06B-SRSS-TB_1x06-1MP_P1.00mm_Vertical, F.Cu at (160.7, 107.1)
- J4: renamed from J5; value EYESPI_Connector -> Conn_EYESPI
- R3: value 732k -> 220k
- R4: value 100k -> 30k
- moved TP4 16.5 mm to (173.8, 91.5)
- moved J4 9.54 mm to (131.3, 105.1)
- moved H3 9.00 mm to (113.5, 107.5)
- moved H4 9.00 mm to (172.5, 107.5)
- moved TP1 4.82 mm to (119.6, 104.4)
- renumbered J4 to J3, J7 to J6, J8 to J7, GND to TP4
Connections:
- A1 pad 10: /CS -> /LITE
- A1 pad 11: /RST -> /DC
- A1 pad 12: /DC -> /RST
- A1 pad 13: /LITE -> /CS
- A1 pad 21: /B_ENCA -> /A_ENCB
- A1 pad 22: /B_ENCB -> /A_ENCA
- A1 pad 25: /A_ENCA -> /B_ENCB
- A1 pad 26: /A_ENCB -> /B_ENCA
Routing:
- net /SCL: track 32.3 -> 11.5 mm
- net /SDA: track 30.5 -> 10.6 mm
- net /CS: track 48.5 -> 29.2 mm, vias 1 -> 0
- net /A_OUT2: track 6.72 -> 25.2 mm
- net /A_OUT1: track 7.08 -> 21.8 mm
- net /RST: track 43.6 -> 29.6 mm, vias 1 -> 0
- net /SCK: track 30.1 -> 19.9 mm, vias 1 -> 2
- net /DC: track 38.9 -> 29.9 mm, vias 1 -> 0
- net /B_ENCA: track 32.6 -> 24.3 mm, vias 1 -> 2
- net /B_ENCB: track 32.1 -> 25.6 mm, vias 0 -> 2
- net /LITE: track 39.5 -> 33.3 mm, vias 1 -> 0
- net +3V3: track 86.2 -> 80.0 mm
- net /MOSI: track 39.4 -> 33.6 mm, vias 1 -> 2
- net GND: track 21.4 -> 24.7 mm, vias 15 -> 17
- net /B_OUT2: track 9.92 -> 12.9 mm
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Other:
- board size 66 x 45 mm -> 66 x 36 mm
- board text removed: "CS"
- board text removed: "DC"
- board text removed: "ENCA"
- board text removed: "ENCB"
- board text removed: "GND"
- board text removed: "LITE"
- board text removed: "M1"
- board text removed: "M2"
- board text removed: "MOSI"
- board text removed: "RST"
- board text removed: "SCK"
- board text removed: "SCL"
- board text removed: "SDA"
- board text removed: "VCC"
