File: hardware/raster-bot/raster-bot.kicad_sch (KiCad schematic)
At the start: 37 parts, among them J1 JUMPER_2PIN, J2 JUMPER_2PIN, J3 PinSocket_1x10, J4 JUMPER_2PIN, J5 EYESPI_Connector, J6 PinSocket_2x06, J7 JST_PH, J8 PinSocket_1x02, SW1 SW_SPDT, U1 DRV8833PWPR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

Commit message: PCB v0.2 update - added motor JST connectors; refactored custom footprints
Parts:
- removed J3: PinSocket_1x10, Connector_PinSocket_2.54mm:PinSocket_1x10_P2.54mm_Vertical, symbol Connector_Generic:Conn_01x10
- removed J6: PinSocket_2x06, Connector_PinSocket_2.54mm:PinSocket_2x06_P2.54mm_Vertical, symbol Connector_Generic:Conn_02x06_Odd_Even
- added J5, J8: Conn_Motor_N20_Encoder, symbol raster-bot:Conn_Motor_N20_Encoder
- J4: renamed from J5; value EYESPI_Connector -> Conn_EYESPI; footprint raster-bot:XUNPU_FPC-05F-18PH20_1x18-1MP_P0.5mm_Horizontal -> (none); symbol raster-bot:EYESPI_Connector -> raster-bot:Conn_EYESPI
- R3: value 732k -> 220k; LCSC C23239 -> C22961
- R4: value 100k -> 30k; LCSC C25803 -> C22984
- renumbered J4 to J3, J7 to J6, J8 to J7
Connections:
- net +3V3: now also J5.4 (VCC), J8.4 (VCC)
- net A_ENCA: now also A1.22 (A3), J5.3 (ENC_A); no longer A1.25 (A6)
- net A_ENCB: now also A1.21 (A2), J5.2 (ENC_B); no longer A1.26 (A7)
- net A_OUT1: now also J5.6 (M1)
- net A_OUT2: now also J5.5 (M2)
- net B_ENCA: now also A1.26 (A7), J8.3 (ENC_A); no longer A1.21 (A2)
- net B_ENCB: now also A1.25 (A6), J8.2 (ENC_B); no longer A1.22 (A3)
- net B_OUT1: now also J8.6 (M1)
- net B_OUT2: now also J8.5 (M2)
- net CS: now also A1.13 (D10/CS); no longer A1.10 (D7)
- net DC: now also A1.11 (D8); no longer A1.12 (D9)
- net GND: now also J5.1 (GND), J8.1 (GND)
- net LITE: now also A1.10 (D7); no longer A1.13 (D10/CS)
- net RST: now also A1.12 (D9); no longer A1.11 (D8)
- no-connect marks 19 -> 22
Other:
- note added: "Touchscreen Connector"
- note removed: "Touchscreen Connectors"
- moved on the sheet: H1, H2, H3, H4
