File: hardware/Raster_Bot/Raster_Bot.kicad_sch (KiCad schematic)
At the start: 37 parts, among them J1 JUMPER_2PIN, J2 JUMPER_2PIN, J3 JUMPER_2PIN, J4 Conn_EYESPI, J5 Conn_Motor_N20_Encoder, J6 JST_PH, J7 PinSocket_1x02, J8 Conn_Motor_N20_Encoder, SW1 SW_SPDT, U1 DRV8833PWPR, U2 TPS61023DRLR

Commit message: Refactor filenames to Raster_Bot
Parts:
- J4: symbol raster-bot:Conn_EYESPI -> Raster_Bot:Conn_EYESPI
- J5, J8: symbol raster-bot:Conn_Motor_N20_Encoder -> Raster_Bot:Conn_Motor_N20_Encoder
- SW1: footprint raster-bot:SW_SPDT_Shouhan_MSK12C02 -> Raster_Bot:SW_SPDT_Shouhan_MSK12C02
- U1: footprint raster-bot:HTSSOP-16-1EP_4.4x5mm_P0.65mm_EP3.4x5mm_Mask2.66x2.46mm_ThermalVias -> Raster_Bot:HTSSOP-16-1EP_4.4x5mm_P0.65mm_EP3.4x5mm_Mask2.66x2.46mm_ThermalVias; symbol raster-bot:DRV8833PWPR -> Raster_Bot:DRV8833PWPR
- U2: symbol raster-bot:TPS61023DRLR -> Raster_Bot:TPS61023DRLR
Changed lines of the file:
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@@
 		)
 		(instances
-			(project "raster-bot"
+			(project "Raster_Bot"
 				(path "/68fd25bc-da1d-4d9a-9340-0ded04d59660"
 					(reference "R2")
@@
 		)
 		(instances
-			(project "raster-bot"
+			(project "Raster_Bot"
 				(path "/68fd25bc-da1d-4d9a-9340-0ded04d59660"
 					(reference "#PWR02")
@@
 		)
 		(instances
-			(project "raster-bot"
+			(project "Raster_Bot"
 				(path "/68fd25bc-da1d-4d9a-9340-0ded04d59660"
 					(reference "#PWR019")
@@
 		)
 		(instances
-			(project "raster-bot"
+			(project "Raster_Bot"
 				(path "/68fd25bc-da1d-4d9a-9340-0ded04d59660"
 					(reference "#PWR021")
@@
 		)
 		(instances
-			(project "raster-bot"
+			(project "Raster_Bot"
 				(path "/68fd25bc-da1d-4d9a-9340-0ded04d59660"
 					(reference "C3")
@@
 		)
 		(instances
-			(project "raster-bot"
+			(project "Raster_Bot"
 				(path "/68fd25bc-da1d-4d9a-9340-0ded04d59660"
 					(reference "H2")
@@
 		)
 		(instances
-			(project "raster-bot"
+			(project "Raster_Bot"
 				(path "/68fd25bc-da1d-4d9a-9340-0ded04d59660"
 					(reference "#PWR024")
@@
 		)
 		(instances
-			(project "raster-bot"
+			(project "Raster_Bot"
 				(path "/68fd25bc-da1d-4d9a-9340-0ded04d59660"
 					(reference "TP1")
@@
 		)
 		(instances
-			(project "raster-bot"
+			(project "Raster_Bot"
 				(path "/68fd25bc-da1d-4d9a-9340-0ded04d59660"
 					(reference "J3")
@@
 		)
 		(instances
-			(project "raster-bot"
+			(project "Raster_Bot"
 				(path "/68fd25bc-da1d-4d9a-9340-0ded04d59660"
 					(reference "H3")
@@
 		)
 		(instances
-			(project "raster-bot"
+			(project "Raster_Bot"
 				(path "/68fd25bc-da1d-4d9a-9340-0ded04d59660"
 					(reference "TP4")
@@
 		)
 		(instances
-			(project "raster-bot"
+			(project "Raster_Bot"
 				(path "/68fd25bc-da1d-4d9a-9340-0ded04d59660"
 					(reference "#PWR07")
@@
 		)
 		(instances
-			(project "raster-bot"
+			(project "Raster_Bot"
 				(path "/68fd25bc-da1d-4d9a-9340-0ded04d59660"
 					(reference "C8")
@@
 		)
 		(instances
-			(project "raster-bot"
+			(project "Raster_Bot"
 				(path "/68fd25bc-da1d-4d9a-9340-0ded04d59660"
 					(reference "#PWR028")
@@
 		)
 		(instances
-			(project "raster-bot"
+			(project "Raster_Bot"
 				(path "/68fd25bc-da1d-4d9a-9340-0ded04d59660"
 					(reference "#PWR026")
@@
 		)
 		(instances
-			(project "raster-bot"
+			(project "Raster_Bot"
 				(path "/68fd25bc-da1d-4d9a-9340-0ded04d59660"
 					(reference "#PWR014")
@@
 		)
 		(instances
-			(project "raster-bot"
+			(project "Raster_Bot"
 				(path "/68fd25bc-da1d-4d9a-9340-0ded04d59660"
 					(reference "#PWR027")
@@
 		)
 		(instances
-			(project "raster-bot"
+			(project "Raster_Bot"
 				(path "/68fd25bc-da1d-4d9a-9340-0ded04d59660"
 					(reference "C7")
@@
 		)
 		(instances
-			(project "raster-bot"
+			(project "Raster_Bot"
 				(path "/68fd25bc-da1d-4d9a-9340-0ded04d59660"
 					(reference "#PWR022")
@@
 		)
 		(instances
-			(project "raster-bot"
+			(project "Raster_Bot"
 				(path "/68fd25bc-da1d-4d9a-9340-0ded04d59660"
 					(reference "R5")
@@
 		)
 		(instances
-			(project "raster-bot"
+			(project "Raster_Bot"
 				(path "/68fd25bc-da1d-4d9a-9340-0ded04d59660"
 					(reference "#PWR010")
@@
 		)
 		(instances
-			(project "raster-bot"
+			(project "Raster_Bot"
 				(path "/68fd25bc-da1d-4d9a-9340-0ded04d59660"
 					(reference "TP2")
@@
 		)
 		(instances
-			(project "raster-bot"
+			(project "Raster_Bot"
 				(path "/68fd25bc-da1d-4d9a-9340-0ded04d59660"
 					(reference "#PWR030")
@@
 		)
 		(instances
-			(project "raster-bot"
+			(project "Raster_Bot"
 				(path "/68fd25bc-da1d-4d9a-9340-0ded04d59660"
 					(reference "#PWR016")
@@
 		)
 		(instances
-			(project "raster-bot"
+			(project "Raster_Bot"
 				(path "/68fd25bc-da1d-4d9a-9340-0ded04d59660"
 					(reference "#PWR017")
@@
 		)
 		(instances
-			(project "raster-bot"
+			(project "Raster_Bot"
 				(path "/68fd25bc-da1d-4d9a-9340-0ded04d59660"
 					(reference "J1")
@@
 		)
 		(instances
-			(project "raster-bot"
+			(project "Raster_Bot"
 				(path "/68fd25bc-da1d-4d9a-9340-0ded04d59660"
 					(reference "#PWR029")
@@
 		)
 		(instances
-			(project "raster-bot"
+			(project "Raster_Bot"
 				(path "/68fd25bc-da1d-4d9a-9340-0ded04d59660"
 					(reference "#PWR020")
@@
 		)
 		(instances
-			(project "raster-bot"
+			(project "Raster_Bot"
 				(path "/68fd25bc-da1d-4d9a-9340-0ded04d59660"
 					(reference "R6")
@@
 		)
 		(instances
-			(project "raster-bot"
+			(project "Raster_Bot"
 				(path "/68fd25bc-da1d-4d9a-9340-0ded04d59660"
 					(reference "R4")
@@
 		)
 		(instances
-			(project "raster-bot"
+			(project "Raster_Bot"
 				(path "/68fd25bc-da1d-4d9a-9340-0ded04d59660"
 					(reference "#PWR03")
@@
 	)
 	(symbol
-		(lib_id "raster-bot:Conn_Motor_N20_Encoder")
+		(lib_id "Raster_Bot:Conn_Motor_N20_Encoder")
 		(at 207.01 134.62 0)
 		(unit 1)
@@
 		)
 		(instances
-			(project "raster-bot"
+			(project "Raster_Bot"
 				(path "/68fd25bc-da1d-4d9a-9340-0ded04d59660"
 					(reference "J8")
@@
 		)
 		(instances
-			(project "raster-bot"
+			(project "Raster_Bot"
 				(path "/68fd25bc-da1d-4d9a-9340-0ded04d59660"
 					(reference "#PWR04")
@@
 	)
 	(symbol
-		(lib_id "raster-bot:TPS61023DRLR")
+		(lib_id "Raster_Bot:TPS61023DRLR")
 		(at 125.73 55.88 0)
 		(unit 1)
@@
 		)
 		(instances
-			(project "raster-bot"
+			(project "Raster_Bot"
 				(path "/68fd25bc-da1d-4d9a-9340-0ded04d59660"
 					(reference "#PWR012")
@@
 		)
 		(instances
-			(project "raster-bot"
+			(project "Raster_Bot"
 				(path "/68fd25bc-da1d-4d9a-9340-0ded04d59660"
 					(reference "#PWR06")
@@
 		)
 		(instances
-			(project "raster-bot"
+			(project "Raster_Bot"
 				(path "/68fd25bc-da1d-4d9a-9340-0ded04d59660"
 					(reference "#PWR05")
@@
 		)
 		(instances
-			(project "raster-bot"
+			(project "Raster_Bot"
 				(path "/68fd25bc-da1d-4d9a-9340-0ded04d59660"
 					(reference "C5")
@@
 		)
 		(instances
-			(project "raster-bot"
+			(project "Raster_Bot"
 				(path "/68fd25bc-da1d-4d9a-9340-0ded04d59660"
 					(reference "C1")
@@
 		)
 		(instances
-			(project "raster-bot"
+			(project "Raster_Bot"
 				(path "/68fd25bc-da1d-4d9a-9340-0ded04d59660"
 					(reference "#FLG02")
@@
 		)
 		(instances
-			(project "raster-bot"
+			(project "Raster_Bot"
 				(path "/68fd25bc-da1d-4d9a-9340-0ded04d59660"
 					(reference "J7")
@@
 		)
 		(instances
-			(project "raster-bot"
+			(project "Raster_Bot"
 				(path "/68fd25bc-da1d-4d9a-9340-0ded04d59660"
 					(reference "D2")
@@
 		)
 		(instances
-			(project "raster-bot"
+			(project "Raster_Bot"
 				(path "/68fd25bc-da1d-4d9a-9340-0ded04d59660"
 					(reference "#PWR08")
@@
 	)
 	(symbol
-		(lib_id "raster-bot:DRV8833PWPR")
+		(lib_id "Raster_Bot:DRV8833PWPR")
 		(at 57.15 153.67 0)
 		(unit 1)
@@
 			)
 		)
-		(property "Footprint" "raster-bot:HTSSOP-16-1EP_4.4x5mm_P0.65mm_EP3.4x5mm_Mask2.66x2.46mm_ThermalVias"
+		(property "Footprint" "Raster_Bot:HTSSOP-16-1EP_4.4x5mm_P0.65mm_EP3.4x5mm_Mask2.66x2.46mm_ThermalVias"
 			(at 62.23 168.91 0)
 			(effects
@@
 		)
 		(instances
-			(project "raster-bot"
+			(project "Raster_Bot"
 				(path "/68fd25bc-da1d-4d9a-9340-0ded04d59660"
 					(reference "#PWR013")
@@
 		)
 		(instances
-			(project "raster-bot"
+			(project "Raster_Bot"
 				(path "/68fd25bc-da1d-4d9a-9340-0ded04d59660"
 					(reference "C2")
@@
 		)
 		(instances
-			(project "raster-bot"
+			(project "Raster_Bot"
 				(path "/68fd25bc-da1d-4d9a-9340-0ded04d59660"
 					(reference "#PWR018")
@@
 		)
 		(instances
-			(project "raster-bot"
+			(project "Raster_Bot"
 				(path "/68fd25bc-da1d-4d9a-9340-0ded04d59660"
 					(reference "J2")
@@
 		)
 		(instances
-			(project "raster-bot"
+			(project "Raster_Bot"
 				(path "/68fd25bc-da1d-4d9a-9340-0ded04d59660"
 					(reference "H4")
@@
 		)
 		(instances
-			(project "raster-bot"
+			(project "Raster_Bot"
 				(path "/68fd25bc-da1d-4d9a-9340-0ded04d59660"
 					(reference "#PWR025")
@@
 		)
 		(instances
-			(project "raster-bot"
+			(project "Raster_Bot"
 				(path "/68fd25bc-da1d-4d9a-9340-0ded04d59660"
 					(reference "#PWR01")
@@
 		)
 		(instances
-			(project "raster-bot"
+			(project "Raster_Bot"
 				(path "/68fd25bc-da1d-4d9a-9340-0ded04d59660"
 					(reference "#PWR011")
@@
 		)
 		(instances
-			(project "raster-bot"
+			(project "Raster_Bot"
 				(path "/68fd25bc-da1d-4d9a-9340-0ded04d59660"
 					(reference "D1")
@@
 		)
 		(instances
-			(project "raster-bot"
+			(project "Raster_Bot"
 				(path "/68fd25bc-da1d-4d9a-9340-0ded04d59660"
 					(reference "C6")
@@
 	(symbol
 		(lib_name "Conn_Motor_N20_Encoder_1")
-		(lib_id "raster-bot:Conn_Motor_N20_Encoder")
+		(lib_id "Raster_Bot:Conn_Motor_N20_Encoder")
 		(at 162.56 134.62 0)
 		(unit 1)
@@
 		)
 		(instances
-			(project "raster-bot"
+			(project "Raster_Bot"
 				(path "/68fd25bc-da1d-4d9a-9340-0ded04d59660"
 					(reference "#PWR015")
@@
 		)
 		(instances
-			(project "raster-bot"
+			(project "Raster_Bot"
 				(path "/68fd25bc-da1d-4d9a-9340-0ded04d59660"
 					(reference "C4")
@@
 	)
 	(symbol
-		(lib_id "raster-bot:Conn_EYESPI")
+		(lib_id "Raster_Bot:Conn_EYESPI")
 		(at 116.84 133.35 0)
 		(unit 1)
@@
 			)
 		)
-		(property "Footprint" "raster-bot:SW_SPDT_Shouhan_MSK12C02"
+		(property "Footprint" "Raster_Bot:SW_SPDT_Shouhan_MSK12C02"
 			(at 203.2 41.91 0)
 			(effects

Commit message: Update hardware design for Raster Bot: modified schematic to include USB-C receptacle, adjusted component properties, and refined sorting options in the project configuration.
Parts:
- removed A1: Arduino_Nano_ESP32, Module:Arduino_Nano, symbol MCU_Module:Arduino_Nano_ESP32
- removed J1, J3: JUMPER_2PIN, Connector_PinHeader_2.54mm:PinHeader_1x02_P2.54mm_Vertical, symbol Connector_Generic:Conn_01x02
- removed SW1: SW_SPDT, Raster_Bot:SW_SPDT_Shouhan_MSK12C02, symbol Switch:SW_SPDT
- removed TP4: TestPoint, TestPoint:TestPoint_Pad_1.5x1.5mm, symbol Connector:TestPoint
- added C1: 1uF, Capacitor_SMD:C_0805_2012Metric, symbol Device:C
- added C2, C8: 0.1uF, Capacitor_SMD:C_0805_2012Metric, symbol Device:C
- added C3: 22uF, Capacitor_SMD:C_0805_2012Metric, symbol Device:C
- added D3: LED, LED_SMD:LED_0603_1608Metric, symbol Device:LED
- added J4: USB_C_Receptacle_USB2.0_16P, symbol Raster_Bot:USB_C_Receptacle_USB2.0_16P
- added R1: 10k, Resistor_SMD:R_0805_2012Metric, symbol Device:R
- added R10: 2.2k, Resistor_SMD:R_0805_2012Metric, symbol Device:R
- added R4, R5: 5.1k, Resistor_SMD:R_0805_2012Metric, symbol Device:R
- added SW1: SW_RESET, Button_Switch_SMD:SW_SPST_TS-1088-xR020, symbol Switch:SW_Push
- added SW2: SW_BOOT, Button_Switch_SMD:SW_SPST_TS-1088-xR020, symbol Switch:SW_Push
- added SW3: SW_SPDT, Raster_Bot:SW_SPDT_Shouhan_MSK12C02, symbol Switch:SW_SPDT
- added U1: ESP32-S3-WROOM-1, RF_Module:ESP32-S3-WROOM-1, symbol RF_Module:ESP32-S3-WROOM-1
- C4: renamed from C1; Voltage 6.3 -> (none)
- C5: renamed from C2; Dielectric X7R -> (none); Voltage 16 -> (none)
- J7: value PinSocket_1x02 -> JUMPER_2PIN; footprint Connector_PinSocket_2.54mm:PinSocket_1x02_P2.54mm_Vertical -> Connector_PinHeader_2.54mm:PinHeader_1x02_P2.54mm_Vertical; LCSC (none) -> C124375; now in the parts list
- R6: renamed from R5; footprint Resistor_SMD:R_0603_1608Metric -> Resistor_SMD:R_0805_2012Metric; LCSC C4190 -> C17520
- R7: renamed from R6; footprint Resistor_SMD:R_0603_1608Metric -> Resistor_SMD:R_0805_2012Metric; LCSC C4190 -> C17520
- R8: renamed from R3; LCSC C22961 -> (none)
- R9: renamed from R4; footprint Resistor_SMD:R_0603_1608Metric -> Resistor_SMD:R_0805_2012Metric; LCSC C22984 -> C17621
- TP1, TP2, TP3: footprint TestPoint:TestPoint_Pad_1.5x1.5mm -> (none); now in the parts list
- renumbered C6 to C10, C7 to C11, C8 to C12, C3 to C6, C4 to C7, C5 to C9, J4 to J1, J5 to J2, J8 to J3, J2 to J5, R1 to R2, R2 to R3, U1 to U2, U2 to U3
Connections:
- net +3V3: now also TP2.1, C2.1, C3.1, R1.1, R10.1, U1.2 (3V3); no longer TP1.1
- net +5V: now also TP3.1; no longer TP2.1
- net CS: now also U1.18 (IO10)
- net DC: now also U1.17 (IO9)
- net GND: now also C1.2, C2.2, C3.2, C8.2, D3.1 (K), J4.A1 (GND), J4.A12 (GND), J4.B1 (GND), J4.B12 (GND), J4.S1 (SHIELD), R4.2, R5.2, SW1.1, SW2.1, U1.1 (GND), U1.40 (GND), U1.41 (GND); no longer J7.2 (Pin_2)
- net LITE: now also U1.7 (IO7)
- net MOSI: now also U1.19 (IO11)
- net RST: now also U1.12 (IO8)
- net SCK: now also U1.20 (IO12)
- net SCL: now also U1.16 (IO46)
- net SDA: now also U1.26 (IO45)
- net SLEEP: now also U1.6 (IO6)
- net at J6.1 (Pin_1): now also SW3.2 (B)
- net +BATT renamed +VBAT
- net +VBAT: now also TP1.1; no longer TP3.1
- net A_ENCA renamed MOT1_ENCA
- net MOT1_ENCA: now also U1.35 (IO42)
- net A_ENCB renamed MOT1_ENCB
- net MOT1_ENCB: now also U1.34 (IO41)
- net A_IN1 renamed MOT1_IN1
- net MOT1_IN1: now also U1.5 (IO5)
- net A_IN2 renamed MOT1_IN2
- net MOT1_IN2: now also U1.4 (IO4)
- net A_OUT1 renamed MOT1_M1
- net A_OUT2 renamed MOT1_M2
- net B_ENCA renamed MOT2_ENCA
- net MOT2_ENCA: now also U1.25 (IO48)
- net B_ENCB renamed MOT2_ENCB
- net MOT2_ENCB: now also U1.24 (IO47)
- net B_IN1 renamed MOT2_IN1
- net MOT2_IN1: now also U1.38 (IO2)
- net B_IN2 renamed MOT2_IN2
- net MOT2_IN2: now also U1.15 (IO3)
- net B_OUT1 renamed MOT2_M1
- net B_OUT2 renamed MOT2_M2
- new net: J7.2 (Pin_2), SW3.1 (A)
- new net: D3.2 (A), R10.2
- new net: J4.A5 (CC1), R5.1
- new net: J4.B5 (CC2), R4.1
- new net +VBUS: J4.A4 (VBUS), J4.A9 (VBUS), J4.B4 (VBUS), J4.B9 (VBUS)
- new net BOOT: SW2.2, U1.27 (IO0)
- new net RESET: C1.1, C8.1, R1.2, SW1.2, U1.3 (EN)
- new net USB_D+: J4.A6 (D+), J4.B6 (D+), U1.14 (USB_D+)
- new net USB_D-: J4.A7 (D-), J4.B7 (D-), U1.13 (USB_D-)
- no-connect marks 22 -> 21
Other:
- note added: "Battery Connector"
- note added: "ESP32-S3-WROOM-1"
- note added: "RESET/BOOT Buttons"
- note added: "Test Points"
- note added: "USB-C Port"
- note removed: "Arduino Nano ESP32"
- note removed: "Battery Input"
- moved on the sheet: C10, C11, C12, C4, C5, C6, C7, C9, D1, D2, H1, H2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

Commit message: [hardware] v0.3 - design upgrade featuring esp32-s3, battery charger, 3.3V LDO, 5V boost coverter
Parts:
- removed C10: 10uF, Capacitor_SMD:C_0805_2012Metric, symbol Device:C
- removed C11: 22uF, Capacitor_SMD:C_0805_2012Metric, symbol Device:C
- removed C9: 0.1uF, Capacitor_SMD:C_0805_2012Metric, symbol Device:C
- removed J7: JUMPER_2PIN, Connector_PinHeader_2.54mm:PinHeader_1x02_P2.54mm_Vertical, symbol Connector_Generic:Conn_01x02
- removed R8: 220k, Resistor_SMD:R_0603_1608Metric, symbol Device:R
- removed R9: 30k, Resistor_SMD:R_0805_2012Metric, symbol Device:R
- removed SW3: SW_SPDT, Raster_Bot:SW_SPDT_Shouhan_MSK12C02, symbol Switch:SW_SPDT
- removed U3: TPS61023DRLR, Package_TO_SOT_SMD:SOT-563, symbol Raster_Bot:TPS61023DRLR
- added C1, C18, C2, C3: 10uF, Capacitor_SMD:C_0805_2012Metric, symbol Device:C
- added C13, C15, C16, C19: 22uF, Capacitor_SMD:C_0805_2012Metric, symbol Device:C
- added C14: 1uF, Capacitor_SMD:C_0603_1608Metric, symbol Device:C
- added C17: 0.1uF, Capacitor_SMD:C_0603_1608Metric, symbol Device:C
- added D1, D2: LED, LED_SMD:LED_0805_2012Metric, symbol Device:LED
- added J8: JUMPER_2PIN, Connector_PinHeader_2.54mm:PinHeader_1x02_P2.54mm_Vertical, symbol Connector_Generic:Conn_01x02
- added Q1: AO3401A, Package_TO_SOT_SMD:SOT-23, symbol Transistor_FET:AO3401A
- added R14, R15: 200k, Resistor_SMD:R_0603_1608Metric, symbol Device:R
- added R16: 100k, Resistor_SMD:R_0603_1608Metric, symbol Device:R
- added R17: 220k, Resistor_SMD:R_0603_1608Metric, symbol Device:R
- added R18: 30k, Resistor_SMD:R_0603_1608Metric, symbol Device:R
- added R3: 1.1k, Resistor_SMD:R_0603_1608Metric, symbol Device:R
- added R4: 2.7k, Resistor_SMD:R_0603_1608Metric, symbol Device:R
- added R5: 10k, Resistor_SMD:R_0603_1608Metric, symbol Device:R
- added R6, R7: 2.2k, Resistor_SMD:R_0603_1608Metric, symbol Device:R
- added SW1: SW_SPDT_SH, Button_Switch_SMD:SW_SPDT_Shouhan_MSK12C02, symbol Raster_Bot:SW_SPDT_SH
- added TP1, TP3: TestPoint, TestPoint:TestPoint_Pad_1.5x1.5mm, symbol Connector:TestPoint
- added U1: BQ24072RGT, Package_DFN_QFN:VQFN-16-1EP_3x3mm_P0.5mm_EP1.6x1.6mm_ThermalVias, symbol Battery_Management:BQ24072RGT
- added U4: AP2114H-3.3, Package_TO_SOT_SMD:SOT-223-3_TabPin2, symbol Raster_Bot:AP2114H-3.3
- added U5: TPS61023DRLR, Package_TO_SOT_SMD:SOT-563, symbol Raster_Bot:TPS61023DRLR
- C10: renamed from C6; footprint Capacitor_SMD:C_0805_2012Metric -> Capacitor_SMD:C_0603_1608Metric; LCSC C28233 -> C14663
- C12: value 22uF -> 10uF; LCSC C45783 -> C15850
- C4: renamed from C1; footprint Capacitor_SMD:C_0805_2012Metric -> Capacitor_SMD:C_0603_1608Metric; LCSC C28323 -> C15849
- C5: renamed from C2; footprint Capacitor_SMD:C_0805_2012Metric -> Capacitor_SMD:C_0603_1608Metric; LCSC C28233 -> C14663
- C7: renamed from C8; footprint Capacitor_SMD:C_0805_2012Metric -> Capacitor_SMD:C_0603_1608Metric; LCSC C28233 -> C14663
- C8: renamed from C4; footprint Capacitor_SMD:C_0805_2012Metric -> Capacitor_SMD:C_0603_1608Metric; LCSC C377773 -> C23630
- C9: renamed from C5; footprint Capacitor_SMD:C_0805_2012Metric -> Capacitor_SMD:C_0603_1608Metric; LCSC C1710 -> C57112
- D3: renamed from D1; footprint LED_SMD:LED_0603_1608Metric -> LED_SMD:LED_0805_2012Metric; LCSC C2286 -> C2297
- D4: renamed from D2; footprint LED_SMD:LED_0603_1608Metric -> LED_SMD:LED_0805_2012Metric; LCSC C2286 -> C2297
- D5: renamed from D3; footprint LED_SMD:LED_0603_1608Metric -> LED_SMD:LED_0805_2012Metric; LCSC C2286 -> C2297
- J2: renamed from J4; footprint (none) -> Raster_Bot:USB_C_Receptacle_G-Switch_GT-USB-7010ASV; LCSC (none) -> C2988369
- J3: renamed from J2; footprint (none) -> Connector_JST:JST_SH_BM06B-SRSS-TB_1x06-1MP_P1.00mm_Vertical
- J4: renamed from J1; footprint (none) -> Raster_Bot:XUNPU_FPC-05F-18PH20_1x18-1MP_P0.5mm_Horizontal
- J5: LCSC C124375 -> C492401
- J6: renamed from J3; footprint (none) -> Connector_JST:JST_SH_BM06B-SRSS-TB_1x06-1MP_P1.00mm_Vertical
- R1: renamed from R4; footprint Resistor_SMD:R_0805_2012Metric -> Resistor_SMD:R_0603_1608Metric; LCSC C27834 -> C23186
- R10: renamed from R7; footprint Resistor_SMD:R_0805_2012Metric -> Resistor_SMD:R_0603_1608Metric; LCSC C17520 -> C4190
- R11: renamed from R10; footprint Resistor_SMD:R_0805_2012Metric -> Resistor_SMD:R_0603_1608Metric; LCSC C17520 -> C4190
- R2: renamed from R5; footprint Resistor_SMD:R_0805_2012Metric -> Resistor_SMD:R_0603_1608Metric; LCSC C27834 -> C23186
- R8: renamed from R1; footprint Resistor_SMD:R_0805_2012Metric -> Resistor_SMD:R_0603_1608Metric; LCSC C17414 -> C25804
- R9: renamed from R6; footprint Resistor_SMD:R_0805_2012Metric -> Resistor_SMD:R_0603_1608Metric; LCSC C17520 -> C4190
- TP2: renamed from TP1; footprint (none) -> TestPoint:TestPoint_Pad_1.5x1.5mm; now left out of the parts list
- TP4: renamed from TP2; footprint (none) -> TestPoint:TestPoint_Pad_1.5x1.5mm; now left out of the parts list
- TP5: renamed from TP3; footprint (none) -> TestPoint:TestPoint_Pad_1.5x1.5mm; now left out of the parts list
- U2: renamed from U1; footprint RF_Module:ESP32-S3-WROOM-1 -> Raster_Bot:ESP32-S3-WROOM-1; LCSC C2913201 -> C2913198
- renumbered C7 to C11, C3 to C6, J6 to J1, R2 to R12, R3 to R13, SW1 to SW2, SW2 to SW3, U2 to U3
Connections:
- net +3V3: now also J4.18 (VCC), C13.1, U4.2 (VO); no longer J4.1 (VCC)
- net +5V: now also C15.1, C16.1, R17.1, U5.6 (VOUT); no longer C12.1, J5.1 (Pin_1), J5.2 (Pin_2)
- net CS: now also J4.10 (DISP_CS), U2.22 (IO14); no longer J4.9 (DISP_CS), U2.18 (IO10)
- net DC: now also J4.12 (DC), U2.20 (IO12); no longer J4.7 (DC), U2.17 (IO9)
- net GND: now also J4.16 (GND), C1.1, C13.2, C14.2, C15.2, C16.2, C17.2, C18.2, C19.1, C2.2, C3.2, R15.2, R18.2, R3.2, R4.2, R5.2, SW1.1 (A), U1.15 (TD), U1.17 (VSS), U1.4 (~{CE}), U1.6 (EN1), U1.8 (VSS), U4.1 (GND), U5.4 (GND); no longer J4.3 (GND)
- net LITE: now also J4.17 (BACKLITE), U2.17 (IO9); no longer J4.2 (BACKLITE), U2.7 (IO7)
- net MOSI: now also J4.14 (MOSI); no longer J4.5 (MOSI)
- net MOT1_ENCA: now also U2.33 (IO40); no longer U2.35 (IO42)
- net MOT1_IN1: now also U2.23 (IO21); no longer U2.5 (IO5)
- net MOT1_IN2: now also U2.24 (IO47); no longer U2.4 (IO4)
- net MOT2_ENCA: now also U2.38 (IO2); no longer U2.25 (IO48)
- net MOT2_ENCB: now also U2.39 (IO1); no longer U2.24 (IO47)
- net MOT2_IN1: now also U2.32 (IO39), U3.10 (BIN2); no longer U2.38 (IO2), U3.9 (BIN1)
- net MOT2_IN2: now also U2.31 (IO38), U3.9 (BIN1); no longer U2.15 (IO3), U3.10 (BIN2)
- net RST: now also J4.11 (RESET), U2.21 (IO13); no longer J4.8 (RESET), U2.12 (IO8)
- net SCK: now also J4.15 (14), U2.18 (IO10); no longer J4.4 (SCK), U2.20 (IO12)
- net SCL: now also J4.6 (SCL), U2.11 (IO18); no longer J4.13 (SCL), U2.16 (IO46)
- net SDA: now also J4.5 (SDA), U2.12 (IO8); no longer J4.14 (SDA), U2.26 (IO45)
- net SLEEP: now also U2.35 (IO42); no longer U2.6 (IO6)
- net VBAT: now reaches J1.1 (Pin_1)
- net VBAT: now also TP2.1, C3.1, R14.1, U1.2 (BAT), U1.3 (BAT)
- net at L1.2: now also U5.5 (SW)
- net CHG: now reaches U2.10 (IO17)
- net CHG: now also D2.1 (K), U1.9 (~{CHG})
- net PGOOD: now reaches U2.9 (IO16)
- net PGOOD: now also D1.1 (K), U1.7 (~{PGOOD})
- removed net +VBAT: L1.1, R9.1, TP2.1
- net +VBUS renamed VBUS
- net VBUS: now also C1.2, TP1.1, U1.13 (IN)
- new net: R5.1, U1.1 (TS)
- new net: Q1.1 (G), R16.2, SW1.2 (B)
- new net: R3.1, U1.12 (ILIM)
- new net: D2.2 (A), R7.2
- new net: R17.2, R18.1, U5.1 (FB)
- new net: D1.2 (A), R6.2
- new net: R4.1, U1.16 (ISET)
- new net VBAT_DIV: C14.1, R14.2, R15.1, U2.7 (IO7)
- new net VSYS: C19.2, J5.1 (Pin_1), J8.1 (Pin_1), Q1.3 (D), R9.1, TP3.1
- new net VSYS_3VIN: C12.1, J5.2 (Pin_2), U4.3 (VI)
- new net VSYS_5VIN: C17.1, C18.1, J8.2 (Pin_2), L1.1, U5.2 (EN), U5.3 (VIN)
- new net VSYS_SRC: C2.1, Q1.2 (S), R16.1, R6.1, R7.1, U1.10 (OUT), U1.11 (OUT), U1.5 (EN2)
- no-connect marks 21 -> 30
Other:
- note added: "3.3V Linear Regulator"
- note added: "Battery Charger"
- note added: "Battery Monitor"
- note added: "ESP32-S3-WROOM-1 N8"
- note added: "Power Switch"
- note added: "no"
- note removed: "ESP32-S3-WROOM-1"
- moved on the sheet: C10, C11, C4, C5, C6, C7, C8, C9, D3, D4, D5, H1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

Commit message: [hardware] Add version silkscreen;
Parts:
- U1: footprint Package_DFN_QFN:VQFN-16-1EP_3x3mm_P0.5mm_EP1.6x1.6mm_ThermalVias -> Raster_Bot:VQFN-16-1EP_3x3mm_P0.5mm_EP1.6x1.6mm_ThermalVias
Changed lines of the file:
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@@
 			)
 		)
-		(property "Footprint" "Package_DFN_QFN:VQFN-16-1EP_3x3mm_P0.5mm_EP1.6x1.6mm_ThermalVias"
+		(property "Footprint" "Raster_Bot:VQFN-16-1EP_3x3mm_P0.5mm_EP1.6x1.6mm_ThermalVias"
 			(at 133.35 82.55 0)
 			(effects
