File: hardware/Raster_Bot/Raster_Bot.kicad_sch (KiCad schematic)
At the start: 67 parts, among them J1 JST_PH, J2 USB_C_Receptacle_USB2.0_16P, J3 Conn_EYESPI, J4 Conn_Motor_N20_Encoder, J5 Conn_Motor_N20_Encoder, Q1 AO3401A, Q2 2N7002, Q3 AO3401A, SW1 SW_RESET, SW2 SW_BOOT, SW3 SW_SPDT_SH, U1 ESP32-S3-MINI-1, U2 BQ24072RGT, U3 DRV8833PWPR, U4 AP2114H-3.3, U5 TPS61023DRLR

Commit message: [hardware] Vendor 3D models locally and upgrade to KiCad 10
Co-authored-by: Cursor <cursoragent@cursor.com>
Parts:
- L1: footprint Inductor_SMD:L_Coilcraft_XxL4030 -> Raster_Bot:L_Coilcraft_XxL4030
- SW3: footprint Button_Switch_SMD:SW_SPDT_Shouhan_MSK12C02 -> Raster_Bot:SW_SPDT_Shouhan_MSK12C02
Changed lines of the file:
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@@
 			)
 		)
-		(property "Footprint" "Button_Switch_SMD:SW_SPDT_Shouhan_MSK12C02"
+		(property "Footprint" "Raster_Bot:SW_SPDT_Shouhan_MSK12C02"
 			(at 181.61 118.11 0)
 			(effects
@@
 			)
 		)
-		(property "Footprint" "Inductor_SMD:L_Coilcraft_XxL4030"
+		(property "Footprint" "Raster_Bot:L_Coilcraft_XxL4030"
 			(at 332.74 36.83 0)
 			(effects
